File: USBC_PD_Trigger_Kicad/V1/USBC_PD_Trigger_Kicad.kicad_sch (KiCad schematic)
At the start: 23 parts, among them J1 USB_C_Receptacle_PowerOnly_6P, J2 Screw_Terminal_01x03, SW1 SW_Push, U1 FUSB302BMPX, U2 ProMicro

Commit message: Added V2 of trigger board w efuse and smaller mc
Parts:
- removed J2: Screw_Terminal_01x03, TerminalBlock_RND:TerminalBlock_RND_205-00046_1x03_P5.00mm_Horizontal, symbol Connector:Screw_Terminal_01x03
- added J2: Screw_Terminal_01x02, TerminalBlock_RND:TerminalBlock_RND_205-00045_1x02_P5.00mm_Horizontal, symbol Connector:Screw_Terminal_01x02
- U1: footprint Package_DFN_QFN:WQFN-14-1EP_2.5x2.5mm_P0.5mm_EP1.45x1.45mm_ThermalVias -> Package_DFN_QFN:WQFN-14-1EP_2.5x2.5mm_P0.5mm_EP1.45x1.45mm
Connections:
- net GND: now also J2.1 (Pin_1)
- net VBUS: now also J2.2 (Pin_2)
Changed lines of the file:
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@@
-	(wire
-		(pts
-			(xy 198.12 93.98) (xy 193.04 93.98)
-		)
-		(stroke
-			(width 0)
-			(type default)
-		)
-	)
 	(wire
 		(pts
@@
 	(wire
 		(pts
-			(xy 181.61 88.9) (xy 198.12 88.9)
-		)
-		(stroke
-			(width 0)
-			(type default)
-		)
-	)
-	(wire
-		(pts
 			(xy 143.51 132.08) (xy 139.7 132.08)
 		)
@@
 	(wire
 		(pts
+			(xy 198.12 91.44) (xy 186.69 91.44)
+		)
+		(stroke
+			(width 0)
+			(type default)
+		)
+	)
+	(wire
+		(pts
 			(xy 81.28 76.2) (xy 72.39 76.2)
 		)
@@
 	(wire
 		(pts
+			(xy 191.77 93.98) (xy 198.12 93.98)
+		)
+		(stroke
+			(width 0)
+			(type default)
+		)
+	)
+	(wire
+		(pts
 			(xy 83.82 116.84) (xy 83.82 114.3)
 		)
@@
 		(pts
 			(xy 80.01 81.28) (xy 80.01 86.36)
-		)
-		(stroke
-			(width 0)
-			(type default)
-		)
-	)
-	(wire
-		(pts
-			(xy 181.61 91.44) (xy 198.12 91.44)
 		)
 		(stroke
@@
 		)
 	)
-	(label "VBUS"
-		(at 181.61 91.44 0)
-		(effects
-			(font
-				(size 1.27 1.27)
-			)
-			(justify left bottom)
-		)
-	)
 	(label "IO4"
 		(at 123.19 129.54 180)
@@
 		)
 	)
-	(label "VCONN"
-		(at 181.61 88.9 0)
+	(label "VBUS"
+		(at 191.77 93.98 0)
 		(effects
 			(font
@@
 			)
 		)
-		(property "Footprint" "Package_DFN_QFN:WQFN-14-1EP_2.5x2.5mm_P0.5mm_EP1.45x1.45mm_ThermalVias"
+		(property "Footprint" "Package_DFN_QFN:WQFN-14-1EP_2.5x2.5mm_P0.5mm_EP1.45x1.45mm"
 			(at 93.98 91.44 0)
 			(effects
@@
 	(symbol
 		(lib_id "power:GND")
-		(at 193.04 93.98 0)
+		(at 186.69 91.44 0)
 		(unit 1)
 		(exclude_from_sim no)
@@
 		(fields_autoplaced yes)
 		(property "Reference" "#PWR011"
-			(at 193.04 100.33 0)
+			(at 186.69 97.79 0)
 			(effects
 				(font
@@
 		)
 		(property "Value" "GND"
-			(at 193.04 99.06 0)
+			(at 186.69 96.52 0)
 			(effects
 				(font
@@
 		)
 		(property "Footprint" ""
-			(at 193.04 93.98 0)
+			(at 186.69 91.44 0)
 			(effects
 				(font
@@
 		)
 		(property "Datasheet" ""
-			(at 193.04 93.98 0)
+			(at 186.69 91.44 0)
 			(effects
 				(font
@@
 		)
 		(property "Description" "Power symbol creates a global label with name \"GND\" , ground"
-			(at 193.04 93.98 0)
+			(at 186.69 91.44 0)
 			(effects
 				(font
@@
 		)
 		(pin "1"
+		)
+		(instances
+			(project "USBC_PD_Trigger_Kicad"
+				(path "/32c0128e-54a9-4266-91fb-d4d3575b4f9a"
+					(reference "#PWR011")
+					(unit 1)
+				)
+			)
+		)
+	)
+	(symbol
+		(lib_id "Connector:Screw_Terminal_01x02")
+		(at 203.2 91.44 0)
+		(unit 1)
+		(exclude_from_sim no)
+		(in_bom yes)
+		(on_board yes)
+		(dnp no)
+		(fields_autoplaced yes)
+		(property "Reference" "J2"
+			(at 205.74 91.4399 0)
+			(effects
+				(font
+					(size 1.27 1.27)
+				)
+				(justify left)
+			)
+		)
+		(property "Value" "Screw_Terminal_01x02"
+			(at 205.74 93.9799 0)
+			(effects
+				(font
+					(size 1.27 1.27)
+				)
+				(justify left)
+			)
+		)
+		(property "Footprint" "TerminalBlock_RND:TerminalBlock_RND_205-00045_1x02_P5.00mm_Horizontal"
+			(at 203.2 91.44 0)
+			(effects
+				(font
+					(size 1.27 1.27)
+				)
+				(hide yes)
+			)
+		)
+		(property "Datasheet" "~"
+			(at 203.2 91.44 0)
+			(effects
+				(font
+					(size 1.27 1.27)
+				)
+				(hide yes)
+			)
+		)
+		(property "Description" "Generic screw terminal, single row, 01x02, script generated (kicad-library-utils/schlib/autogen/connector/)"
+			(at 203.2 91.44 0)
+			(effects
+				(font
+					(size 1.27 1.27)
+				)
+				(hide yes)
+			)
+		)
+		(pin "1"
+		)
+		(pin "2"
 		)
 		(instances
 			(project ""
 				(path "/32c0128e-54a9-4266-91fb-d4d3575b4f9a"
-					(reference "#PWR011")
+					(reference "J2")
 					(unit 1)
 				)
@@
 					(unit 1)
 				)
-			)
-		)
-	)
-	(symbol
-		(lib_id "Connector:Screw_Terminal_01x03")
-		(at 203.2 91.44 0)
-		(unit 1)
-		(exclude_from_sim no)
-		(in_bom yes)
-		(on_board yes)
-		(dnp no)
-		(fields_autoplaced yes)
-		(property "Reference" "J2"
-			(at 205.74 90.1699 0)
-			(effects
-				(font
-					(size 1.27 1.27)
-				)
-				(justify left)
-			)
-		)
-		(property "Value" "Screw_Terminal_01x03"
-			(at 205.74 92.7099 0)
-			(effects
-				(font
-					(size 1.27 1.27)
-				)
-				(justify left)
-			)
-		)
-		(property "Footprint" "TerminalBlock_RND:TerminalBlock_RND_205-00046_1x03_P5.00mm_Horizontal"
-			(at 203.2 91.44 0)
-			(effects
-				(font
-					(size 1.27 1.27)
-				)
-				(hide yes)
-			)
-		)
-		(property "Datasheet" "~"
-			(at 203.2 91.44 0)
-			(effects
-				(font
-					(size 1.27 1.27)
-				)
-				(hide yes)
-			)
-		)
-		(property "Description" "Generic screw terminal, single row, 01x03, script generated (kicad-library-utils/schlib/autogen/connector/)"
-			(at 203.2 91.44 0)
-			(effects
-				(font
-					(size 1.27 1.27)
-				)
-				(hide yes)
-			)
-		)
-		(pin "1"
-		)
-		(pin "2"
-		)
-		(pin "3"
-		)
-		(instances
-			(project ""
-				(path "/32c0128e-54a9-4266-91fb-d4d3575b4f9a"
-					(reference "J2")
-					(unit 1)
-				)
